File: Stepdown led board.kicad_sch (KiCad schematic)
At the start: 5 parts, among them J1 In, J2 Out, J3 Stepdown

Commit message: - Fixed dumb stepdown module inversion - Fixed Front silkscreen
Connections:
- net +12V: now also J3.2 (Pin_2); no longer J3.3 (Pin_3)
- net GND: now also J3.3 (Pin_3); no longer J3.2 (Pin_2)
- net Vout: now also J3.4 (Pin_4); no longer J3.1 (Pin_1)
Changed lines of the file:
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@@
   (junction (at 26.67 21.59) (diameter 0) (color 0 0 0 0)
   )
-  (no_connect (at 71.12 27.94))
+  (no_connect (at 69.85 20.32))
   (wire (pts (xy 48.26 21.59) (xy 48.26 17.78))
-    (stroke (width 0) (type default) (color 0 0 0 0))
-  )
-  (wire (pts (xy 71.12 27.94) (xy 73.66 27.94))
     (stroke (width 0) (type default) (color 0 0 0 0))
   )
@@
     (stroke (width 0) (type default) (color 0 0 0 0))
   )
+  (wire (pts (xy 69.85 22.86) (xy 73.66 22.86))
+    (stroke (width 0) (type default) (color 0 0 0 0))
+  )
   (wire (pts (xy 73.66 45.72) (xy 68.58 45.72))
     (stroke (width 0) (type default) (color 0 0 0 0))
   )
+  (wire (pts (xy 69.85 27.94) (xy 73.66 27.94))
+    (stroke (width 0) (type default) (color 0 0 0 0))
+  )
   (wire (pts (xy 48.26 17.78) (xy 26.67 17.78))
+    (stroke (width 0) (type default) (color 0 0 0 0))
+  )
+  (wire (pts (xy 69.85 20.32) (xy 73.66 20.32))
     (stroke (width 0) (type default) (color 0 0 0 0))
   )
@@
     (stroke (width 0) (type default) (color 0 0 0 0))
   )
-  (wire (pts (xy 69.85 25.4) (xy 73.66 25.4))
-    (stroke (width 0) (type default) (color 0 0 0 0))
-  )
-  (wire (pts (xy 69.85 22.86) (xy 73.66 22.86))
-    (stroke (width 0) (type default) (color 0 0 0 0))
-  )
-  (wire (pts (xy 66.04 20.32) (xy 73.66 20.32))
-    (stroke (width 0) (type default) (color 0 0 0 0))
-  )
   (wire (pts (xy 73.66 36.83) (xy 68.58 36.83))
     (stroke (width 0) (type default) (color 0 0 0 0))
   )
   (wire (pts (xy 25.4 21.59) (xy 26.67 21.59))
+    (stroke (width 0) (type default) (color 0 0 0 0))
+  )
+  (wire (pts (xy 69.85 25.4) (xy 73.66 25.4))
     (stroke (width 0) (type default) (color 0 0 0 0))
   )
@@
     )
   )
-  (global_label "Vout" (shape output) (at 66.04 20.32 180) (fields_autoplaced)
+  (global_label "Vout" (shape output) (at 69.85 27.94 180) (fields_autoplaced)
     (effects (font (size 1.27 1.27)) (justify right))
-    (property "Intersheet References" "${INTERSHEET_REFS}" (id 0) (at 59.5145 20.2406 0)
+    (property "Intersheet References" "${INTERSHEET_REFS}" (id 0) (at 63.3245 27.8606 0)
       (effects (font (size 1.27 1.27)) (justify right) hide)
     )
@@
     (pin "3")
   )
-  (symbol (lib_id "power:+12V") (at 69.85 25.4 90) (unit 1)
+  (symbol (lib_id "power:+12V") (at 69.85 22.86 90) (unit 1)
     (in_bom yes) (on_board yes) (fields_autoplaced)
-    (property "Reference" "#PWR0105" (id 0) (at 73.66 25.4 0)
+    (property "Reference" "#PWR0105" (id 0) (at 73.66 22.86 0)
       (effects (font (size 1.27 1.27)) hide)
     )
-    (property "Value" "+12V" (id 1) (at 66.04 25.3999 90)
+    (property "Value" "+12V" (id 1) (at 66.04 22.8599 90)
       (effects (font (size 1.27 1.27)) (justify left))
     )
-    (property "Footprint" "" (id 2) (at 69.85 25.4 0)
+    (property "Footprint" "" (id 2) (at 69.85 22.86 0)
       (effects (font (size 1.27 1.27)) hide)
     )
-    (property "Datasheet" "" (id 3) (at 69.85 25.4 0)
+    (property "Datasheet" "" (id 3) (at 69.85 22.86 0)
       (effects (font (size 1.27 1.27)) hide)
     )
@@
     (pin "2")
   )
-  (symbol (lib_id "power:GND") (at 69.85 22.86 270) (unit 1)
+  (symbol (lib_id "power:GND") (at 69.85 25.4 270) (unit 1)
     (in_bom yes) (on_board yes) (fields_autoplaced)
-    (property "Reference" "#PWR0104" (id 0) (at 63.5 22.86 0)
+    (property "Reference" "#PWR0104" (id 0) (at 63.5 25.4 0)
       (effects (font (size 1.27 1.27)) hide)
     )
-    (property "Value" "GND" (id 1) (at 66.04 22.8599 90)
+    (property "Value" "GND" (id 1) (at 66.04 25.3999 90)
       (effects (font (size 1.27 1.27)) (justify right))
     )
-    (property "Footprint" "" (id 2) (at 69.85 22.86 0)
+    (property "Footprint" "" (id 2) (at 69.85 25.4 0)
       (effects (font (size 1.27 1.27)) hide)
     )
-    (property "Datasheet" "" (id 3) (at 69.85 22.86 0)
+    (property "Datasheet" "" (id 3) (at 69.85 25.4 0)
       (effects (font (size 1.27 1.27)) hide)
     )
